File: LFO1.sch (KiCad schematic (older format))
At the start: 20 parts, among them P1 100k, P2 100k, U1 4XOPAMP

Commit message: added README.md
Parts:
- C1: Type (none) -> Polystyrene
- C2, C3: renamed from C?; Type (none) -> Ceramic
- D1, D2, D3, D4: renamed from R?; Type (none) -> Signal Diode
- R1, R2: renamed from 4k7; value RES -> 4k7; Tolerance (none) -> 1%; Type (none) -> Metal Film
- R3: renamed from R1; Tolerance (none) -> 1%; Type (none) -> Metal Film
- R4, R6, R7: renamed from R?; Tolerance (none) -> 1%; Type (none) -> Metal Film
- R5: renamed from 10k; value RES -> 10k; Tolerance (none) -> 1%; Type (none) -> Metal Film
- gave numbers to parts that had none: 1
Changed lines of the file:
@@
-EESchema Schematic File Version 2  date Sun 17 Nov 2013 14:47:36 GMT
+EESchema Schematic File Version 2  date Wed 20 Nov 2013 17:13:23 GMT
 LIBS:power
 LIBS:device
@@
 LIBS:-15v
 LIBS:gnd
-LIBS:FreakSynth101-cache
 EELAYER 25  0
 EELAYER END
@@
 Sheet 1 1
 Title ""
-Date "27 oct 2013"
+Date "20 nov 2013"
 Rev ""
 Comp ""
@@
 $EndComp
 $Comp
-L CAP C?
+L CAP C3
 U 1 1 5248A205
 P 2800 3425
-F 0 "C?" H 2850 3525 50  0000 L CNN
+F 0 "C3" H 2850 3525 50  0000 L CNN
 F 1 "100nF" H 2850 3325 50  0000 L CNN
+F 4 "Ceramic" H 2800 3425 60  0001 C CNN "Type"
 	1    2800 3425
 	-1   0    0    1
 $EndComp
 $Comp
-L CAP C?
+L CAP C2
 U 1 1 5248A1E6
 P 2800 2950
-F 0 "C?" H 2850 3050 50  0000 L CNN
+F 0 "C2" H 2850 3050 50  0000 L CNN
 F 1 "100nF" H 2850 2850 50  0000 L CNN
+F 4 "Ceramic" H 2800 2950 60  0001 C CNN "Type"
 	1    2800 2950
 	-1   0    0    1
@@
 $EndComp
 $Comp
-L RES R?
+L RES R7
 U 1 1 52486C35
 P 8000 4125
-F 0 "R?" H 8000 4025 50  0000 C CNN
+F 0 "R7" H 8000 4025 50  0000 C CNN
 F 1 "1k" H 7995 4225 50  0000 C CNN
+F 4 "Metal Film" H 8000 4125 60  0001 C CNN "Type"
+F 5 "1%" H 8000 4125 60  0001 C CNN "Tolerance"
 	1    8000 4125
 	1    0    0    -1
 $EndComp
 $Comp
-L LED D?
+L LED D5
 U 1 1 52486BFE
 P 7425 4125
-F 0 "D?" H 7425 4225 50  0000 C CNN
+F 0 "D5" H 7425 4225 50  0000 C CNN
 F 1 "LED" H 7425 4025 50  0000 C CNN
 	1    7425 4125
@@
 $EndComp
 $Comp
-L RES R?
+L RES R6
 U 1 1 524867EB
 P 6600 4600
-F 0 "R?" H 6600 4500 50  0000 C CNN
+F 0 "R6" H 6600 4500 50  0000 C CNN
 F 1 "10k" H 6595 4700 50  0000 C CNN
+F 4 "Metal Film" H 6600 4600 60  0001 C CNN "Type"
+F 5 "1%" H 6600 4600 60  0001 C CNN "Tolerance"
 	1    6600 4600
 	1    0    0    -1
 $EndComp
 $Comp
-L RES 10k
+L RES R5
 U 1 1 524867B5
 P 6200 4175
-F 0 "10k" H 6200 4075 50  0000 C CNN
-F 1 "RES" H 6195 4275 50  0000 C CNN
+F 0 "R5" H 6200 4075 50  0000 C CNN
+F 1 "10k" H 6195 4275 50  0000 C CNN
+F 4 "Metal Film" H 6200 4175 60  0001 C CNN "Type"
+F 5 "1%" H 6200 4175 60  0001 C CNN "Tolerance"
 	1    6200 4175
 	0    1    1    0
@@
 SHAPE\n
 $Comp
-L RES 4k7
+L RES R2
 U 1 1 52484E79
 P 4550 4450
-F 0 "4k7" H 4550 4350 50  0000 C CNN
-F 1 "RES" H 4545 4550 50  0000 C CNN
+F 0 "R2" H 4550 4350 50  0000 C CNN
+F 1 "4k7" H 4545 4550 50  0000 C CNN
+F 4 "Metal Film" H 4550 4450 60  0001 C CNN "Type"
+F 5 "1%" H 4550 4450 60  0001 C CNN "Tolerance"
 	1    4550 4450
 	1    0    0    -1
 $EndComp
 $Comp
-L RES 4k7
+L RES R1
 U 1 1 52484E6F
 P 4550 3650
-F 0 "4k7" H 4550 3550 50  0000 C CNN
-F 1 "RES" H 4545 3750 50  0000 C CNN
+F 0 "R1" H 4550 3550 50  0000 C CNN
+F 1 "4k7" H 4545 3750 50  0000 C CNN
+F 4 "Metal Film" H 4550 3650 60  0001 C CNN "Type"
+F 5 "1%" H 4550 3650 60  0001 C CNN "Tolerance"
 	1    4550 3650
 	1    0    0    -1
@@
 F 0 "C1" H 5800 3300 50  0000 L CNN
 F 1 "470nF" H 5800 3100 50  0000 L CNN
+F 4 "Polystyrene" H 5750 3200 60  0001 C CNN "Type"
 	1    5750 3200
 	0    1    1    0
@@
 $EndComp
 $Comp
-L RES R?
+L RES R4
 U 1 1 524702D7
 P 7400 3200
-F 0 "R?" H 7400 3100 50  0000 C CNN
+F 0 "R4" H 7400 3100 50  0000 C CNN
 F 1 "10k" H 7395 3300 50  0000 C CNN
+F 4 "Metal Film" H 7400 3200 60  0001 C CNN "Type"
+F 5 "1%" H 7400 3200 60  0001 C CNN "Tolerance"
 	1    7400 3200
 	1    0    0    -1
 $EndComp
 $Comp
-L RES R1
+L RES R3
 U 1 1 524702C6
 P 6600 3200
-F 0 "R1" H 6600 3100 50  0000 C CNN
+F 0 "R3" H 6600 3100 50  0000 C CNN
 F 1 "3k9" H 6595 3300 50  0000 C CNN
+F 4 "Metal Film" H 6600 3200 60  0001 C CNN "Type"
+F 5 "1%" H 6600 3200 60  0001 C CNN "Tolerance"
 	1    6600 3200
 	1    0    0    -1
 $EndComp
 $Comp
-L SIGNAL_DIODE R?
+L SIGNAL_DIODE D1
 U 1 1 524701E8
 P 3125 4725
-F 0 "R?" H 3125 4575 50  0000 C CNN
+F 0 "D1" H 3125 4575 50  0000 C CNN
 F 1 "1N4148" H 3120 4875 50  0000 C CNN
+F 4 "Signal Diode" H 3125 4725 60  0001 C CNN "Type"
 	1    3125 4725
 	0    1    -1   0
 $EndComp
 $Comp
-L SIGNAL_DIODE R?
+L SIGNAL_DIODE D2
 U 1 1 524701E4
 P 3550 4700
-F 0 "R?" H 3550 4550 50  0000 C CNN
+F 0 "D2" H 3550 4550 50  0000 C CNN
 F 1 "1N4148" H 3545 4850 50  0000 C CNN
+F 4 "Signal Diode" H 3550 4700 60  0001 C CNN "Type"
 	1    3550 4700
 	0    1    1    0
@@
 $EndComp
 $Comp
-L SIGNAL_DIODE R?
+L SIGNAL_DIODE D4
 U 1 1 5246FFAB
 P 5100 4450
-F 0 "R?" H 5100 4300 50  0000 C CNN
+F 0 "D4" H 5100 4300 50  0000 C CNN
 F 1 "1N4148" H 5095 4600 50  0000 C CNN
+F 4 "Signal Diode" H 5100 4450 60  0001 C CNN "Type"
 	1    5100 4450
 	-1   0    0    1
 $EndComp
 $Comp
-L SIGNAL_DIODE R?
+L SIGNAL_DIODE D3
 U 1 1 5246FF9A
 P 5100 3650
-F 0 "R?" H 5100 3500 50  0000 C CNN
+F 0 "D3" H 5100 3500 50  0000 C CNN
 F 1 "1N4148" H 5095 3800 50  0000 C CNN
+F 4 "Signal Diode" H 5100 3650 60  0001 C CNN "Type"
 	1    5100 3650
 	1    0    0    -1
